File: V1/PCB/PhotonButtons.brd (EAGLE design)
At the start: 70 x 37 mm, 25 parts, among them Q1 MOSFET-NCHANNEL2N7002PW

Commit message: Added components values
Parts:
- D1, D2: value BAT20J -> 1SS355TE-17
- R3, R6, R7: value (none) -> 100k
Changed lines of the file:
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@@
 <setting verticaltext="up"/>
 </settings>
-<grid distance="0.025" unitdist="inch" unit="inch" style="lines" multiple="1" display="no" altdistance="0.006" altunitdist="inch" altunit="inch"/>
+<grid distance="0.1" unitdist="mm" unit="mm" style="lines" multiple="1" display="no" altdistance="0.006" altunitdist="inch" altunit="inch"/>
 <layers>
 <layer number="1" name="Top" color="4" fill="1" visible="no" active="yes"/>
@@
 <vertex x="26.67" y="33.655"/>
 </polygon>
+<dimension x1="4" y1="4" x2="66" y2="4" x3="35" y3="-2.2" textsize="1.27" textratio="16" layer="47"/>
+<dimension x1="66" y1="4" x2="66" y2="33" x3="73.5" y3="18.5" textsize="1.27" textratio="16" layer="47"/>
 </plain>
 <attributes>
@@
 </autorouter>
 <elements>
-<element name="D1" library="SparkFun-DiscreteSemi" package="SOD-323" value="BAT20J" x="16.5354" y="24.7142" smashed="yes" rot="R180">
+<element name="D1" library="SparkFun-DiscreteSemi" package="SOD-323" value="1SS355TE-17" x="16.5354" y="24.7142" smashed="yes" rot="R180">
 <attribute name="PROD_ID" value="DIO-11623" x="16.5354" y="24.7142" size="1.778" layer="27" rot="R180" display="off"/>
 <attribute name="NAME" x="20.1168" y="25.146" size="1.016" layer="25" rot="R180"/>
-</element>
-<element name="D2" library="SparkFun-DiscreteSemi" package="SOD-323" value="BAT20J" x="16.51" y="22.86" smashed="yes" rot="R180">
+<attribute name="FARNELL" value="152-5435" x="16.5354" y="24.7142" size="1.778" layer="27" rot="R180" display="off"/>
+</element>
+<element name="D2" library="SparkFun-DiscreteSemi" package="SOD-323" value="1SS355TE-17" x="16.51" y="22.86" smashed="yes" rot="R180">
 <attribute name="PROD_ID" value="DIO-11623" x="16.51" y="22.86" size="1.778" layer="27" rot="R180" display="off"/>
 <attribute name="NAME" x="20.1168" y="23.4696" size="1.016" layer="25" rot="R180"/>
 <attribute name="VALUE" x="17.526" y="21.971" size="0.4064" layer="27" rot="R180"/>
+<attribute name="FARNELL" value="152-5435" x="16.51" y="22.86" size="1.778" layer="27" rot="R180" display="off"/>
 </element>
 <element name="FRAME1" library="SparkFun-Aesthetics" package="CREATIVE_COMMONS" value="FRAME-LETTER" x="20.955" y="-11.43"/>
@@
 <attribute name="VALUE" x="19.2786" y="16.4338" size="0.4064" layer="27" rot="R90"/>
 </element>
-<element name="R6" library="SparkFun-Resistors" package="0805" value="" x="48.895" y="13.97" smashed="yes" rot="R270">
+<element name="R6" library="SparkFun-Resistors" package="0805" value="100k" x="48.895" y="13.97" smashed="yes" rot="R270">
 <attribute name="NAME" x="48.26" y="15.748" size="1.016" layer="25"/>
 <attribute name="VALUE" x="47.371" y="15.367" size="0.4064" layer="27" rot="R270"/>
 </element>
-<element name="R7" library="SparkFun-Resistors" package="0805" value="" x="14.2875" y="4.7625" smashed="yes">
+<element name="R7" library="SparkFun-Resistors" package="0805" value="100k" x="14.2875" y="4.7625" smashed="yes">
 <attribute name="NAME" x="13.0175" y="5.9055" size="1.016" layer="25"/>
 <attribute name="VALUE" x="12.8905" y="3.2385" size="0.4064" layer="27"/>
@@
 <attribute name="PROD_ID" value="TRANS-11151" x="14.5796" y="17.0942" size="1.778" layer="27" rot="R270" display="off"/>
 <attribute name="NAME" x="13.7843" y="18.4388" size="1.016" layer="25"/>
+<attribute name="FARNELL" value="189-4713" x="14.5796" y="17.0942" size="1.778" layer="27" rot="R270" display="off"/>
 </element>
 <element name="R2" library="SparkFun-Resistors" package="0805" value="1M" x="20.955" y="13.97" smashed="yes" rot="R90">
@@
 <element name="LOGO2" library="SparkFun-Aesthetics" package="OSHW-LOGO-L" value="OSHW-LOGOL" x="63.476" y="25" rot="MR0"/>
 <element name="H3" library="holes" package="3,2" value="MOUNT-HOLE3.2" x="66" y="33"/>
-<element name="R3" library="SparkFun-Resistors" package="0805" value="" x="21.59" y="26.67" smashed="yes" rot="R90">
+<element name="R3" library="SparkFun-Resistors" package="0805" value="100k" x="21.59" y="26.67" smashed="yes" rot="R90">
 <attribute name="NAME" x="20.8788" y="28.4607" size="1.016" layer="25"/>
 <attribute name="VALUE" x="22.987" y="25.654" size="0.4064" layer="27" rot="R90"/>
